Commit message: Fixed navigation

File: src/descriptions/amr_combo_v2/urdf/amr_combo_v2.urdf.xacro (robot description, xacro)
@@ -92,5 +92,5 @@
         </link>
         <joint
-            name="base_footprint"
+            name="base_footprint_joint"
             type="fixed">
             <origin
@@ -98,7 +98,7 @@
                 rpy="0 0 0" />
             <parent
-                link="base_link" />
-            <child
                 link="base_footprint" />
+            <child
+                link="base_link" />
             <axis
                 xyz="0 0 0" />
@@ -144,24 +144,15 @@
             </collision>
         </link>
+        <!-- These joint needs to be fixed since n plugin for Gazebo -->
         <joint
             name="mpo_700_caster_back_left_joint"
-            type="revolute">
+            type="fixed">
             <origin
                 xyz="-0.26 0.26 0.22"
                 rpy="0 0 0" />
             <parent
-                link="base_footprint" />
+                link="base_link" />
             <child
                 link="mpo_700_caster_back_left_link" />
-            <axis
-                xyz="0 0 1" />
-            <limit
-                lower="-1E+16"
-                upper="1E+16"
-                effort="1000"
-                velocity="6.5" />
-            <dynamics
-                damping="30"
-                friction="110" />
         </joint>
         <link
@@ -207,5 +198,5 @@
         <joint
             name="mpo_700_wheel_back_left_joint"
-            type="revolute">
+            type="fixed">
             <origin
                 xyz="0 -0.0453 -0.122"
@@ -215,14 +206,4 @@
             <child
                 link="mpo_700_wheel_back_left_link" />
-            <axis
-                xyz="0 1 0" />
-            <limit
-                lower="-1E+16"
-                upper="1E+16"
-                effort="1000"
-                velocity="20.5" />
-            <dynamics
-                damping="30"
-                friction="110" />
         </joint>
         <link
@@ -268,22 +249,12 @@
         <joint
             name="mpo_700_caster_back_right_joint"
-            type="revolute">
+            type="fixed">
             <origin
                 xyz="-0.26 -0.26 0.22"
                 rpy="0 0 0" />
             <parent
-                link="base_footprint" />
+                link="base_link" />
             <child
                 link="mpo_700_caster_back_right_link" />
-            <axis
-                xyz="0 0 1" />
-            <limit
-                lower="-1E+16"
-                upper="1E+16"
-                effort="1000"
-                velocity="6.5" />
-            <dynamics
-                damping="30"
-                friction="110" />
         </joint>
         <link
@@ -329,5 +300,5 @@
         <joint
             name="mpo_700_wheel_back_right_joint"
-            type="revolute">
+            type="fixed">
             <origin
                 xyz="0 -0.0453 -0.122"
@@ -337,14 +308,4 @@
             <child
                 link="mpo_700_wheel_back_right_link" />
-            <axis
-                xyz="0 -1 0" />
-            <limit
-                lower="-1E+16"
-                upper="1E+16"
-                effort="1000"
-                velocity="20.5" />
-            <dynamics
-                damping="30"
-                friction="110" />
         </joint>
         <link
@@ -390,22 +351,12 @@
         <joint
             name="mpo_700_caster_front_left_joint"
-            type="revolute">
+            type="fixed">
             <origin
                 xyz="0.26 0.26 0.22"
                 rpy="0 0 0" />
             <parent
-                link="base_footprint" />
+                link="base_link" />
             <child
                 link="mpo_700_caster_front_left_link" />
-            <axis
-                xyz="0 0 1" />
-            <limit
-                lower="-1E+16"
-                upper="1E+16"
-                effort="1000"
-                velocity="6.5" />
-            <dynamics
-                damping="30"
-                friction="110" />
         </joint>
         <link
@@ -451,5 +402,5 @@
         <joint
             name="mpo_700_wheel_front_left_joint"
-            type="revolute">
+            type="fixed">
             <origin
                 xyz="0 -0.0453 -0.122"
@@ -459,14 +410,4 @@
             <child
                 link="mpo_700_wheel_front_left_link" />
-            <axis
-                xyz="0 1 0" />
-            <limit
-                lower="-1E+16"
-                upper="1E+16"
-                effort="10000"
-                velocity="20.5" />
-            <dynamics
-                damping="30"
-                friction="110" />
         </joint>
         <link
@@ -512,22 +453,12 @@
         <joint
             name="mpo_700_caster_front_right_joint"
-            type="revolute">
+            type="fixed">
             <origin
                 xyz="0.26 -0.26 0.22"
                 rpy="0 0 0" />
             <parent
-                link="base_footprint" />
+                link="base_link" />
             <child
                 link="mpo_700_caster_front_right_link" />
-            <axis
-                xyz="0 0 1" />
-            <limit
-                lower="-1E+16"
-                upper="1E+16"
-                effort="1000"
-                velocity="6.5" />
-            <dynamics
-                damping="30"
-                friction="110" />
         </joint>
         <link
@@ -573,5 +504,5 @@
         <joint
             name="mpo_700_wheel_front_right_joint"
-            type="revolute">
+            type="fixed">
             <origin
                 xyz="0 -0.0453 -0.122"
@@ -581,14 +512,4 @@
             <child
                 link="mpo_700_wheel_front_right_link" />
-            <axis
-                xyz="0 -1 0" />
-            <limit
-                lower="-1E+16"
-                upper="1E+16"
-                effort="1000"
-                velocity="20.5" />
-            <dynamics
-                damping="30"
-                friction="110" />
         </joint>
         <link
