Commit message: Updated base (2->3) and awtube (18kg_v2->3)

File: src/awcombo_moveit_config/config/awcombo.ros2_control.xacro (robot description, xacro)
@@ -8,43 +8,43 @@
                 <plugin>mock_components/GenericSystem</plugin>
             </hardware>
-            <joint name="awtube2_18kg_v2_joint1">
+            <joint name="awtube_joint1">
                 <command_interface name="position"/>
                 <state_interface name="position">
-                  <param name="initial_value">${initial_positions['awtube2_18kg_v2_joint1']}</param>
+                  <param name="initial_value">${initial_positions['awtube_joint1']}</param>
                 </state_interface>
                 <state_interface name="velocity"/>
             </joint>
-            <joint name="awtube2_18kg_v2_joint2">
+            <joint name="awtube_joint2">
                 <command_interface name="position"/>
                 <state_interface name="position">
-                  <param name="initial_value">${initial_positions['awtube2_18kg_v2_joint2']}</param>
+                  <param name="initial_value">${initial_positions['awtube_joint2']}</param>
                 </state_interface>
                 <state_interface name="velocity"/>
             </joint>
-            <joint name="awtube2_18kg_v2_joint3">
+            <joint name="awtube_joint3">
                 <command_interface name="position"/>
                 <state_interface name="position">
-                  <param name="initial_value">${initial_positions['awtube2_18kg_v2_joint3']}</param>
+                  <param name="initial_value">${initial_positions['awtube_joint3']}</param>
                 </state_interface>
                 <state_interface name="velocity"/>
             </joint>
-            <joint name="awtube2_18kg_v2_joint4">
+            <joint name="awtube_joint4">
                 <command_interface name="position"/>
                 <state_interface name="position">
-                  <param name="initial_value">${initial_positions['awtube2_18kg_v2_joint4']}</param>
+                  <param name="initial_value">${initial_positions['awtube_joint4']}</param>
                 </state_interface>
                 <state_interface name="velocity"/>
             </joint>
-            <joint name="awtube2_18kg_v2_joint5">
+            <joint name="awtube_joint5">
                 <command_interface name="position"/>
                 <state_interface name="position">
-                  <param name="initial_value">${initial_positions['awtube2_18kg_v2_joint5']}</param>
+                  <param name="initial_value">${initial_positions['awtube_joint5']}</param>
                 </state_interface>
                 <state_interface name="velocity"/>
             </joint>
-            <joint name="awtube2_18kg_v2_joint6">
+            <joint name="awtube_joint6">
                 <command_interface name="position"/>
                 <state_interface name="position">
-                  <param name="initial_value">${initial_positions['awtube2_18kg_v2_joint6']}</param>
+                  <param name="initial_value">${initial_positions['awtube_joint6']}</param>
                 </state_interface>
                 <state_interface name="velocity"/>

File: src/descriptions/awcombo_description/urdf/awcombo.xacro (robot description, xacro)
@@ -6,7 +6,7 @@
     <xacro:arg name="iname" default="eno1" />
     <!-- Amr combo base -->
-    <xacro:include filename="$(find amr_combo_v2)/urdf/amr_combo_v2.urdf.xacro"/>
+    <xacro:include filename="$(find amr_combo_v3)/urdf/amr_combo_v3.urdf.xacro"/>
     <!-- Robotic arm -->
-    <xacro:include filename="$(find awtube2_18kg_v2)/urdf/awtube2_18kg_v2.urdf.xacro" />
+    <xacro:include filename="$(find awtube31814v2)/xacro/awtube31814v2.xacro" />
     <!-- Gripper -->
     <xacro:include filename="$(find grip_exon)/urdf/grip_exon.urdf.xacro" />
@@ -18,12 +18,12 @@
     <xacro:include filename="$(find awcombo_description)/urdf/awtube.ros2_control.xacro" />
     <!-- Calling the macros, starting from neo base -->
-    <xacro:amr_combo_v2 name="base_footprint" parent="base_link">
+    <xacro:amr_combo_v3 name="base_footprint" parent="base_link">
         <origin xyz="0 0 0" rpy="0 0 0" />
-    </xacro:amr_combo_v2>
-    <xacro:awtube2_18kg_v2 parent="agv_link1">
-        <origin xyz="0 0 0" rpy="0 0 0" />
-    </xacro:awtube2_18kg_v2>
-    <xacro:grip_exon parent="awtube2_18kg_v2_link6">
-        <origin xyz="0 0 0.057" rpy="0 0 -1.57" />
+    </xacro:amr_combo_v3>
+    <xacro:awtube3 connected_to="agv_link1">
+        <origin xyz="0 0 0" rpy="0 0 1.57" />
+    </xacro:awtube3>
+    <xacro:grip_exon parent="awtube_link6">
+        <origin xyz="0 0 0.0" rpy="0 0 -1.57" />
     </xacro:grip_exon>
     <xacro:camera_support parent="GRIPPER">

File: src/descriptions/awcombo_description/urdf/awtube.ros2_control.xacro (robot description, xacro)
@@ -66,5 +66,5 @@
             </gpio> -->
             <!-- Joints -->
-            <joint name="awtube2_18kg_v2_joint1">
+            <joint name="awtube_joint1">
                 <command_interface name="position" />
                 <!-- <command_interface name="velocity" />
@@ -79,5 +79,5 @@
                 </ec_module> -->
             </joint>
-            <joint name="awtube2_18kg_v2_joint2">
+            <joint name="awtube_joint2">
                 <command_interface name="position" />
                 <!-- <command_interface name="velocity" />
@@ -92,5 +92,5 @@
                 </ec_module> -->
             </joint>
-            <joint name="awtube2_18kg_v2_joint3">
+            <joint name="awtube_joint3">
                 <command_interface name="position" />
                 <!-- <command_interface name="velocity" />
@@ -105,5 +105,5 @@
                 </ec_module> -->
             </joint>
-            <joint name="awtube2_18kg_v2_joint4">
+            <joint name="awtube_joint4">
                 <command_interface name="position" />
                 <!-- <command_interface name="velocity" />
@@ -118,5 +118,5 @@
                 </ec_module> -->
             </joint>
-            <joint name="awtube2_18kg_v2_joint5">
+            <joint name="awtube_joint5">
                 <command_interface name="position" />
                 <!-- <command_interface name="velocity" />
@@ -131,5 +131,5 @@
                 </ec_module> -->
             </joint>
-            <joint name="awtube2_18kg_v2_joint6">
+            <joint name="awtube_joint6">
                 <command_interface name="position" />
                 <!-- <command_interface name="velocity" />
